Commit message: `hubero_bringup_gazebo_ros` & gazebo - skin file in the `spawn_actor.launch` made configurable [#59]

File: hubero_gazebo/urdf/actor.xacro (robot description, xacro)
@@ -13,4 +13,5 @@
     <xacro:arg name="pose_yaw" default="-1.5707" />
     <xacro:arg name="visualize_laser" default="false" />
+    <xacro:arg name="skin_file" default="walk.dae" />
     <!-- Arg->Property hack from PMB2 description -->
     <xacro:property name="actor_name" value="$(arg actor_name)" />
@@ -22,8 +23,9 @@
     <xacro:property name="pose_yaw" value="$(arg pose_yaw)" />
     <xacro:property name="visualize_laser" value="$(arg visualize_laser)" />
+    <xacro:property name="skin_file" value="$(arg skin_file)" />
     <actor name="${actor_name}">
         <pose>${pose_x} ${pose_y} ${pose_z} ${pose_roll} ${pose_pitch} ${pose_yaw}</pose>
         <skin>
-            <filename>walk.dae</filename>
+            <filename>${skin_file}</filename>
             <scale>1.0</scale>
         </skin>
